File: hardware/pi3a-prototype/electrical/base/interfaces.kicad_sch (KiCad schematic)
At the start: 4 parts, among them J1 J1 interface, J100 J100 interface, J101 J101 interface, J102 J102 interface

Commit message: feat(hardware): figer le checkpoint D1-3 et sa reprise en pause
Parts:
- J101: footprint (none) -> NATHAN_USB:Power_Pigtail_2Pad
- J102: footprint (none) -> Connector_JST:JST_PH_B3B-PH-K_1x03_P2.00mm_Vertical
Connections:
- net USB_CHARGE_RUN: now reaches J1.29 (Pin_29)
- net USB_CHARGE_CLOCK: now reaches J1.31 (Pin_31)
- no-connect marks 17 -> 15
Changed lines of the file:
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@@
 (no_connect (at 312.42 52.07))
 (no_connect (at 312.42 54.61))
-(no_connect (at 312.42 57.15))
+(wire (pts (xy 312.42 57.15) (xy 320.04 57.15)) (stroke (width 0) (type default)))
+(global_label "USB_CHARGE_RUN" (shape bidirectional) (at 320.04 57.15 180) (effects (font (size 0.9 0.9))) (property "Intersheetrefs" "${INTERSHEET_REFS}" (at 320.04 57.15 180) (effects (font (size 0.9 0.9)) hide)))
 (wire (pts (xy 312.42 59.69) (xy 320.04 59.69)) (stroke (width 0) (type default)))
 (global_label "GND" (shape bidirectional) (at 320.04 59.69 180) (effects (font (size 0.9 0.9))) (property "Intersheetrefs" "${INTERSHEET_REFS}" (at 320.04 59.69 180) (effects (font (size 0.9 0.9)) hide)))
-(no_connect (at 312.42 62.23))
+(wire (pts (xy 312.42 62.23) (xy 320.04 62.23)) (stroke (width 0) (type default)))
+(global_label "USB_CHARGE_CLOCK" (shape bidirectional) (at 320.04 62.23 180) (effects (font (size 0.9 0.9))) (property "Intersheetrefs" "${INTERSHEET_REFS}" (at 320.04 62.23 180) (effects (font (size 0.9 0.9)) hide)))
 (no_connect (at 312.42 64.77))
 (no_connect (at 312.42 67.31))
@@
 (wire (pts (xy 312.42 85.09) (xy 320.04 85.09)) (stroke (width 0) (type default)))
 (global_label "I2S_DOUT" (shape bidirectional) (at 320.04 85.09 180) (effects (font (size 0.9 0.9))) (property "Intersheetrefs" "${INTERSHEET_REFS}" (at 320.04 85.09 180) (effects (font (size 0.9 0.9)) hide)))
-(symbol (lib_id "NATHAN:J101") (at 487.68 60.96 0) (unit 1) (in_bom yes) (on_board yes) (dnp no) (property "Reference" "J101" (at 487.68 53.15 0) (effects (font (size 1.2 1.2)))) (property "Value" "J101 interface" (at 487.68 68.77 0) (effects (font (size 1 1)))) (property "Footprint" "" (at 487.68 60.96 0) (effects (font (size 1 1)) hide)) (pin "1")(pin "2") (instances (project "nathan-base" (path "/136d3303-0d33-56a8-b18c-a25e8527c00a/8c3930c7-591f-56b4-9278-3340fcffa2a3" (reference "J101") (unit 1)))))
+(symbol (lib_id "NATHAN:J101") (at 487.68 60.96 0) (unit 1) (in_bom yes) (on_board yes) (dnp no) (property "Reference" "J101" (at 487.68 53.15 0) (effects (font (size 1.2 1.2)))) (property "Value" "J101 interface" (at 487.68 68.77 0) (effects (font (size 1 1)))) (property "Footprint" "NATHAN_USB:Power_Pigtail_2Pad" (at 487.68 60.96 0) (effects (font (size 1 1)) hide)) (pin "1")(pin "2") (instances (project "nathan-base" (path "/136d3303-0d33-56a8-b18c-a25e8527c00a/8c3930c7-591f-56b4-9278-3340fcffa2a3" (reference "J101") (unit 1)))))
 (wire (pts (xy 469.9 60.96) (xy 462.28 60.96)) (stroke (width 0) (type default)))
 (global_label "5V_SYS" (shape bidirectional) (at 462.28 60.96 0) (effects (font (size 0.9 0.9))) (property "Intersheetrefs" "${INTERSHEET_REFS}" (at 462.28 60.96 0) (effects (font (size 0.9 0.9)) hide)))
 (wire (pts (xy 505.46 60.96) (xy 513.08 60.96)) (stroke (width 0) (type default)))
 (global_label "GND" (shape bidirectional) (at 513.08 60.96 180) (effects (font (size 0.9 0.9))) (property "Intersheetrefs" "${INTERSHEET_REFS}" (at 513.08 60.96 180) (effects (font (size 0.9 0.9)) hide)))
-(symbol (lib_id "NATHAN:J102") (at 680.72 60.96 0) (unit 1) (in_bom yes) (on_board yes) (dnp no) (property "Reference" "J102" (at 680.72 53.15 0) (effects (font (size 1.2 1.2)))) (property "Value" "J102 interface" (at 680.72 68.77 0) (effects (font (size 1 1)))) (property "Footprint" "" (at 680.72 60.96 0) (effects (font (size 1 1)) hide)) (pin "1")(pin "2")(pin "3") (instances (project "nathan-base" (path "/136d3303-0d33-56a8-b18c-a25e8527c00a/8c3930c7-591f-56b4-9278-3340fcffa2a3" (reference "J102") (unit 1)))))
+(symbol (lib_id "NATHAN:J102") (at 680.72 60.96 0) (unit 1) (in_bom yes) (on_board yes) (dnp no) (property "Reference" "J102" (at 680.72 53.15 0) (effects (font (size 1.2 1.2)))) (property "Value" "J102 interface" (at 680.72 68.77 0) (effects (font (size 1 1)))) (property "Footprint" "Connector_JST:JST_PH_B3B-PH-K_1x03_P2.00mm_Vertical" (at 680.72 60.96 0) (effects (font (size 1 1)) hide)) (pin "1")(pin "2")(pin "3") (instances (project "nathan-base" (path "/136d3303-0d33-56a8-b18c-a25e8527c00a/8c3930c7-591f-56b4-9278-3340fcffa2a3" (reference "J102") (unit 1)))))
 (wire (pts (xy 662.94 59.69) (xy 655.32 59.69)) (stroke (width 0) (type default)))
 (global_label "I2C_SDA" (shape bidirectional) (at 655.32 59.69 0) (effects (font (size 0.9 0.9))) (property "Intersheetrefs" "${INTERSHEET_REFS}" (at 655.32 59.69 0) (effects (font (size 0.9 0.9)) hide)))
@@
 (wire (pts (xy 698.5 59.69) (xy 706.12 59.69)) (stroke (width 0) (type default)))
 (global_label "GND" (shape bidirectional) (at 706.12 59.69 180) (effects (font (size 0.9 0.9))) (property "Intersheetrefs" "${INTERSHEET_REFS}" (at 706.12 59.69 180) (effects (font (size 0.9 0.9)) hide)))
+(symbol (lib_id "NATHAN:#FLG1") (at 101.6 127 0) (unit 1) (in_bom no) (on_board no) (dnp no) (property "Reference" "#FLG1" (at 101.6 119.19 0) (effects (font (size 1.2 1.2)))) (property "Value" "PWR_FLAG" (at 101.6 134.81 0) (effects (font (size 1 1)))) (property "Footprint" "" (at 101.6 127 0) (effects (font (size 1 1)) hide)) (pin "1") (instances (project "nathan-base" (path "/136d3303-0d33-56a8-b18c-a25e8527c00a/8c3930c7-591f-56b4-9278-3340fcffa2a3" (reference "#FLG1") (unit 1)))))
+(wire (pts (xy 83.82 127) (xy 76.2 127)) (stroke (width 0) (type default)))
+(global_label "5V_SYS" (shape bidirectional) (at 76.2 127 0) (effects (font (size 0.9 0.9))) (property "Intersheetrefs" "${INTERSHEET_REFS}" (at 76.2 127 0) (effects (font (size 0.9 0.9)) hide)))
+(symbol (lib_id "NATHAN:#FLG2") (at 294.64 127 0) (unit 1) (in_bom no) (on_board no) (dnp no) (property "Reference" "#FLG2" (at 294.64 119.19 0) (effects (font (size 1.2 1.2)))) (property "Value" "PWR_FLAG" (at 294.64 134.81 0) (effects (font (size 1 1)))) (property "Footprint" "" (at 294.64 127 0) (effects (font (size 1 1)) hide)) (pin "1") (instances (project "nathan-base" (path "/136d3303-0d33-56a8-b18c-a25e8527c00a/8c3930c7-591f-56b4-9278-3340fcffa2a3" (reference "#FLG2") (unit 1)))))
+(wire (pts (xy 276.86 127) (xy 269.24 127)) (stroke (width 0) (type default)))
+(global_label "3V3_PI" (shape bidirectional) (at 269.24 127 0) (effects (font (size 0.9 0.9))) (property "Intersheetrefs" "${INTERSHEET_REFS}" (at 269.24 127 0) (effects (font (size 0.9 0.9)) hide)))
+(symbol (lib_id "NATHAN:#FLG3") (at 487.68 127 0) (unit 1) (in_bom no) (on_board no) (dnp no) (property "Reference" "#FLG3" (at 487.68 119.19 0) (effects (font (size 1.2 1.2)))) (property "Value" "PWR_FLAG" (at 487.68 134.81 0) (effects (font (size 1 1)))) (property "Footprint" "" (at 487.68 127 0) (effects (font (size 1 1)) hide)) (pin "1") (instances (project "nathan-base" (path "/136d3303-0d33-56a8-b18c-a25e8527c00a/8c3930c7-591f-56b4-9278-3340fcffa2a3" (reference "#FLG3") (unit 1)))))
+(wire (pts (xy 469.9 127) (xy 462.28 127)) (stroke (width 0) (type default)))
+(global_label "GND" (shape bidirectional) (at 462.28 127 0) (effects (font (size 0.9 0.9))) (property "Intersheetrefs" "${INTERSHEET_REFS}" (at 462.28 127 0) (effects (font (size 0.9 0.9)) hide)))
+(symbol (lib_id "NATHAN:#FLG4") (at 680.72 127 0) (unit 1) (in_bom no) (on_board no) (dnp no) (property "Reference" "#FLG4" (at 680.72 119.19 0) (effects (font (size 1.2 1.2)))) (property "Value" "PWR_FLAG" (at 680.72 134.81 0) (effects (font (size 1 1)))) (property "Footprint" "" (at 680.72 127 0) (effects (font (size 1 1)) hide)) (pin "1") (instances (project "nathan-base" (path "/136d3303-0d33-56a8-b18c-a25e8527c00a/8c3930c7-591f-56b4-9278-3340fcffa2a3" (reference "#FLG4") (unit 1)))))
+(wire (pts (xy 662.94 127) (xy 655.32 127)) (stroke (width 0) (type default)))
+(global_label "USB_PC_VBUS" (shape bidirectional) (at 655.32 127 0) (effects (font (size 0.9 0.9))) (property "Intersheetrefs" "${INTERSHEET_REFS}" (at 655.32 127 0) (effects (font (size 0.9 0.9)) hide)))
 )
