File: hardware/pi3a-prototype/electrical/base/nathan-base.kicad_sch (KiCad schematic)
At the start: 0 parts

Commit message: feat(hardware): figer le checkpoint D1-3 et sa reprise en pause
Other:
- removed sheet audio-boundary
- removed sheet usb-boundary
- added sheet audio-dac (audio-dac.kicad_sch)
- added sheet audio-filter (audio-filter.kicad_sch)
- added sheet audio-headphone (audio-headphone.kicad_sch)
- added sheet audio-power (audio-power.kicad_sch)
- added sheet usb-data (usb-data.kicad_sch)
- added sheet usb-detect (usb-detect.kicad_sch)
- added sheet usb-policy (usb-policy.kicad_sch)
- added sheet usb-port (usb-port.kicad_sch)
- added sheet usb-power-legacy (usb-power-legacy.kicad_sch)
- added sheet usb-power-typec (usb-power-typec.kicad_sch)
- note added: "D1 proposal: see validation/native-current for revision-specific evidence. Component and manufacturing qualification pending."
- note removed: "D1 proposal: see validation/native-current for ERC evidence. USB/audio boundaries unresolved; no fabrication approval."
