File: hardware/pi3a-prototype/electrical/controls/analog.kicad_sch (KiCad schematic)
At the start: 19 parts, among them J20 J20 interface, J21 J21 interface, J22 J22 interface, J23 J23 interface, U6 MCP3208-CI/SL

Commit message: feat(hardware): figer le checkpoint D1-3 et sa reprise en pause
Parts:
- J20, J21: footprint (none) -> Connector_JST:JST_PH_B5B-PH-K_1x05_P2.00mm_Vertical
- J22, J23: footprint (none) -> Connector_JST:JST_PH_B3B-PH-K_1x03_P2.00mm_Vertical
Changed lines of the file:
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@@
 (wire (pts (xy 505.46 259.08) (xy 513.08 259.08)) (stroke (width 0) (type default)))
 (global_label "GND" (shape bidirectional) (at 513.08 259.08 180) (effects (font (size 0.9 0.9))) (property "Intersheetrefs" "${INTERSHEET_REFS}" (at 513.08 259.08 180) (effects (font (size 0.9 0.9)) hide)))
-(symbol (lib_id "NATHAN:J20") (at 680.72 259.08 0) (unit 1) (in_bom yes) (on_board yes) (dnp no) (property "Reference" "J20" (at 680.72 250 0) (effects (font (size 1.2 1.2)))) (property "Value" "J20 interface" (at 680.72 268.16 0) (effects (font (size 1 1)))) (property "Footprint" "" (at 680.72 259.08 0) (effects (font (size 1 1)) hide)) (pin "1")(pin "2")(pin "3")(pin "4")(pin "5") (instances (project "nathan-controls" (path "/2f5d4a0a-9476-5e3c-a978-b6f76052ad70/d169995f-4bc5-51f5-ae04-4808cddc92f7" (reference "J20") (unit 1)))))
+(symbol (lib_id "NATHAN:J20") (at 680.72 259.08 0) (unit 1) (in_bom yes) (on_board yes) (dnp no) (property "Reference" "J20" (at 680.72 250 0) (effects (font (size 1.2 1.2)))) (property "Value" "J20 interface" (at 680.72 268.16 0) (effects (font (size 1 1)))) (property "Footprint" "Connector_JST:JST_PH_B5B-PH-K_1x05_P2.00mm_Vertical" (at 680.72 259.08 0) (effects (font (size 1 1)) hide)) (pin "1")(pin "2")(pin "3")(pin "4")(pin "5") (instances (project "nathan-controls" (path "/2f5d4a0a-9476-5e3c-a978-b6f76052ad70/d169995f-4bc5-51f5-ae04-4808cddc92f7" (reference "J20") (unit 1)))))
 (wire (pts (xy 662.94 256.54) (xy 655.32 256.54)) (stroke (width 0) (type default)))
 (global_label "3V3_PI" (shape bidirectional) (at 655.32 256.54 0) (effects (font (size 0.9 0.9))) (property "Intersheetrefs" "${INTERSHEET_REFS}" (at 655.32 256.54 0) (effects (font (size 0.9 0.9)) hide)))
@@
 (wire (pts (xy 698.5 259.08) (xy 706.12 259.08)) (stroke (width 0) (type default)))
 (global_label "STICK_L_CLICK" (shape bidirectional) (at 706.12 259.08 180) (effects (font (size 0.9 0.9))) (property "Intersheetrefs" "${INTERSHEET_REFS}" (at 706.12 259.08 180) (effects (font (size 0.9 0.9)) hide)))
-(symbol (lib_id "NATHAN:J21") (at 101.6 325.12 0) (unit 1) (in_bom yes) (on_board yes) (dnp no) (property "Reference" "J21" (at 101.6 316.04 0) (effects (font (size 1.2 1.2)))) (property "Value" "J21 interface" (at 101.6 334.2 0) (effects (font (size 1 1)))) (property "Footprint" "" (at 101.6 325.12 0) (effects (font (size 1 1)) hide)) (pin "1")(pin "2")(pin "3")(pin "4")(pin "5") (instances (project "nathan-controls" (path "/2f5d4a0a-9476-5e3c-a978-b6f76052ad70/d169995f-4bc5-51f5-ae04-4808cddc92f7" (reference "J21") (unit 1)))))
+(symbol (lib_id "NATHAN:J21") (at 101.6 325.12 0) (unit 1) (in_bom yes) (on_board yes) (dnp no) (property "Reference" "J21" (at 101.6 316.04 0) (effects (font (size 1.2 1.2)))) (property "Value" "J21 interface" (at 101.6 334.2 0) (effects (font (size 1 1)))) (property "Footprint" "Connector_JST:JST_PH_B5B-PH-K_1x05_P2.00mm_Vertical" (at 101.6 325.12 0) (effects (font (size 1 1)) hide)) (pin "1")(pin "2")(pin "3")(pin "4")(pin "5") (instances (project "nathan-controls" (path "/2f5d4a0a-9476-5e3c-a978-b6f76052ad70/d169995f-4bc5-51f5-ae04-4808cddc92f7" (reference "J21") (unit 1)))))
 (wire (pts (xy 83.82 322.58) (xy 76.2 322.58)) (stroke (width 0) (type default)))
 (global_label "3V3_PI" (shape bidirectional) (at 76.2 322.58 0) (effects (font (size 0.9 0.9))) (property "Intersheetrefs" "${INTERSHEET_REFS}" (at 76.2 322.58 0) (effects (font (size 0.9 0.9)) hide)))
@@
 (wire (pts (xy 119.38 325.12) (xy 127 325.12)) (stroke (width 0) (type default)))
 (global_label "STICK_R_CLICK" (shape bidirectional) (at 127 325.12 180) (effects (font (size 0.9 0.9))) (property "Intersheetrefs" "${INTERSHEET_REFS}" (at 127 325.12 180) (effects (font (size 0.9 0.9)) hide)))
-(symbol (lib_id "NATHAN:J22") (at 294.64 325.12 0) (unit 1) (in_bom yes) (on_board yes) (dnp no) (property "Reference" "J22" (at 294.64 317.31 0) (effects (font (size 1.2 1.2)))) (property "Value" "J22 interface" (at 294.64 332.93 0) (effects (font (size 1 1)))) (property "Footprint" "" (at 294.64 325.12 0) (effects (font (size 1 1)) hide)) (pin "1")(pin "2")(pin "3") (instances (project "nathan-controls" (path "/2f5d4a0a-9476-5e3c-a978-b6f76052ad70/d169995f-4bc5-51f5-ae04-4808cddc92f7" (reference "J22") (unit 1)))))
+(symbol (lib_id "NATHAN:J22") (at 294.64 325.12 0) (unit 1) (in_bom yes) (on_board yes) (dnp no) (property "Reference" "J22" (at 294.64 317.31 0) (effects (font (size 1.2 1.2)))) (property "Value" "J22 interface" (at 294.64 332.93 0) (effects (font (size 1 1)))) (property "Footprint" "Connector_JST:JST_PH_B3B-PH-K_1x03_P2.00mm_Vertical" (at 294.64 325.12 0) (effects (font (size 1 1)) hide)) (pin "1")(pin "2")(pin "3") (instances (project "nathan-controls" (path "/2f5d4a0a-9476-5e3c-a978-b6f76052ad70/d169995f-4bc5-51f5-ae04-4808cddc92f7" (reference "J22") (unit 1)))))
 (wire (pts (xy 276.86 323.85) (xy 269.24 323.85)) (stroke (width 0) (type default)))
 (global_label "3V3_PI" (shape bidirectional) (at 269.24 323.85 0) (effects (font (size 0.9 0.9))) (property "Intersheetrefs" "${INTERSHEET_REFS}" (at 269.24 323.85 0) (effects (font (size 0.9 0.9)) hide)))
@@
 (wire (pts (xy 312.42 323.85) (xy 320.04 323.85)) (stroke (width 0) (type default)))
 (global_label "RAW_L2" (shape bidirectional) (at 320.04 323.85 180) (effects (font (size 0.9 0.9))) (property "Intersheetrefs" "${INTERSHEET_REFS}" (at 320.04 323.85 180) (effects (font (size 0.9 0.9)) hide)))
-(symbol (lib_id "NATHAN:J23") (at 487.68 325.12 0) (unit 1) (in_bom yes) (on_board yes) (dnp no) (property "Reference" "J23" (at 487.68 317.31 0) (effects (font (size 1.2 1.2)))) (property "Value" "J23 interface" (at 487.68 332.93 0) (effects (font (size 1 1)))) (property "Footprint" "" (at 487.68 325.12 0) (effects (font (size 1 1)) hide)) (pin "1")(pin "2")(pin "3") (instances (project "nathan-controls" (path "/2f5d4a0a-9476-5e3c-a978-b6f76052ad70/d169995f-4bc5-51f5-ae04-4808cddc92f7" (reference "J23") (unit 1)))))
+(symbol (lib_id "NATHAN:J23") (at 487.68 325.12 0) (unit 1) (in_bom yes) (on_board yes) (dnp no) (property "Reference" "J23" (at 487.68 317.31 0) (effects (font (size 1.2 1.2)))) (property "Value" "J23 interface" (at 487.68 332.93 0) (effects (font (size 1 1)))) (property "Footprint" "Connector_JST:JST_PH_B3B-PH-K_1x03_P2.00mm_Vertical" (at 487.68 325.12 0) (effects (font (size 1 1)) hide)) (pin "1")(pin "2")(pin "3") (instances (project "nathan-controls" (path "/2f5d4a0a-9476-5e3c-a978-b6f76052ad70/d169995f-4bc5-51f5-ae04-4808cddc92f7" (reference "J23") (unit 1)))))
 (wire (pts (xy 469.9 323.85) (xy 462.28 323.85)) (stroke (width 0) (type default)))
 (global_label "3V3_PI" (shape bidirectional) (at 462.28 323.85 0) (effects (font (size 0.9 0.9))) (property "Intersheetrefs" "${INTERSHEET_REFS}" (at 462.28 323.85 0) (effects (font (size 0.9 0.9)) hide)))
