File: hardware/pi3a-prototype/electrical/controls/digital.kicad_sch (KiCad schematic)
At the start: 28 parts, among them J24 J24 interface, J25 J25 interface, SW10 B3F-4055 candidate, SW11 B3F-4055 candidate, SW2 B3F-4055 candidate, SW3 B3F-4055 candidate, SW4 B3F-4055 candidate, SW5 B3F-4055 candidate, SW6 B3F-4055 candidate, SW7 B3F-4055 candidate, SW8 B3F-4055 candidate, SW9 B3F-4055 candidate, U7 MCP23017-E/SO

Commit message: feat(hardware): figer le checkpoint D1-3 et sa reprise en pause
Parts:
- J24, J25: footprint (none) -> Connector_JST:JST_PH_B2B-PH-K_1x02_P2.00mm_Vertical
Changed lines of the file:
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@@
 (wire (pts (xy 312.42 457.2) (xy 320.04 457.2)) (stroke (width 0) (type default)))
 (global_label "3V3_PI" (shape bidirectional) (at 320.04 457.2 180) (effects (font (size 0.9 0.9))) (property "Intersheetrefs" "${INTERSHEET_REFS}" (at 320.04 457.2 180) (effects (font (size 0.9 0.9)) hide)))
-(symbol (lib_id "NATHAN:J24") (at 487.68 457.2 0) (unit 1) (in_bom yes) (on_board yes) (dnp no) (property "Reference" "J24" (at 487.68 449.39 0) (effects (font (size 1.2 1.2)))) (property "Value" "J24 interface" (at 487.68 465.01 0) (effects (font (size 1 1)))) (property "Footprint" "" (at 487.68 457.2 0) (effects (font (size 1 1)) hide)) (pin "1")(pin "2") (instances (project "nathan-controls" (path "/2f5d4a0a-9476-5e3c-a978-b6f76052ad70/335e8db8-b1a3-55fa-81b5-5d0597f4b273" (reference "J24") (unit 1)))))
+(symbol (lib_id "NATHAN:J24") (at 487.68 457.2 0) (unit 1) (in_bom yes) (on_board yes) (dnp no) (property "Reference" "J24" (at 487.68 449.39 0) (effects (font (size 1.2 1.2)))) (property "Value" "J24 interface" (at 487.68 465.01 0) (effects (font (size 1 1)))) (property "Footprint" "Connector_JST:JST_PH_B2B-PH-K_1x02_P2.00mm_Vertical" (at 487.68 457.2 0) (effects (font (size 1 1)) hide)) (pin "1")(pin "2") (instances (project "nathan-controls" (path "/2f5d4a0a-9476-5e3c-a978-b6f76052ad70/335e8db8-b1a3-55fa-81b5-5d0597f4b273" (reference "J24") (unit 1)))))
 (wire (pts (xy 469.9 457.2) (xy 462.28 457.2)) (stroke (width 0) (type default)))
 (global_label "SHOULDER_L1" (shape bidirectional) (at 462.28 457.2 0) (effects (font (size 0.9 0.9))) (property "Intersheetrefs" "${INTERSHEET_REFS}" (at 462.28 457.2 0) (effects (font (size 0.9 0.9)) hide)))
 (wire (pts (xy 505.46 457.2) (xy 513.08 457.2)) (stroke (width 0) (type default)))
 (global_label "GND" (shape bidirectional) (at 513.08 457.2 180) (effects (font (size 0.9 0.9))) (property "Intersheetrefs" "${INTERSHEET_REFS}" (at 513.08 457.2 180) (effects (font (size 0.9 0.9)) hide)))
-(symbol (lib_id "NATHAN:J25") (at 680.72 457.2 0) (unit 1) (in_bom yes) (on_board yes) (dnp no) (property "Reference" "J25" (at 680.72 449.39 0) (effects (font (size 1.2 1.2)))) (property "Value" "J25 interface" (at 680.72 465.01 0) (effects (font (size 1 1)))) (property "Footprint" "" (at 680.72 457.2 0) (effects (font (size 1 1)) hide)) (pin "1")(pin "2") (instances (project "nathan-controls" (path "/2f5d4a0a-9476-5e3c-a978-b6f76052ad70/335e8db8-b1a3-55fa-81b5-5d0597f4b273" (reference "J25") (unit 1)))))
+(symbol (lib_id "NATHAN:J25") (at 680.72 457.2 0) (unit 1) (in_bom yes) (on_board yes) (dnp no) (property "Reference" "J25" (at 680.72 449.39 0) (effects (font (size 1.2 1.2)))) (property "Value" "J25 interface" (at 680.72 465.01 0) (effects (font (size 1 1)))) (property "Footprint" "Connector_JST:JST_PH_B2B-PH-K_1x02_P2.00mm_Vertical" (at 680.72 457.2 0) (effects (font (size 1 1)) hide)) (pin "1")(pin "2") (instances (project "nathan-controls" (path "/2f5d4a0a-9476-5e3c-a978-b6f76052ad70/335e8db8-b1a3-55fa-81b5-5d0597f4b273" (reference "J25") (unit 1)))))
 (wire (pts (xy 662.94 457.2) (xy 655.32 457.2)) (stroke (width 0) (type default)))
 (global_label "SHOULDER_R1" (shape bidirectional) (at 655.32 457.2 0) (effects (font (size 0.9 0.9))) (property "Intersheetrefs" "${INTERSHEET_REFS}" (at 655.32 457.2 0) (effects (font (size 0.9 0.9)) hide)))
