File: hardware/pi3a-prototype/electrical/controls/haptic-5.kicad_sch (KiCad schematic)
At the start: 6 parts, among them J6 J6 interface, U5 DRV2604LDGSR

Commit message: feat(hardware): figer le checkpoint D1-3 et sa reprise en pause
Parts:
- J6: footprint (none) -> Connector_JST:JST_PH_B2B-PH-K_1x02_P2.00mm_Vertical
Changed lines of the file:
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@@
 (wire (pts (xy 119.38 127) (xy 127 127)) (stroke (width 0) (type default)))
 (global_label "3V3_HAPTIC" (shape bidirectional) (at 127 127 180) (effects (font (size 0.9 0.9))) (property "Intersheetrefs" "${INTERSHEET_REFS}" (at 127 127 180) (effects (font (size 0.9 0.9)) hide)))
-(symbol (lib_id "NATHAN:J6") (at 294.64 127 0) (unit 1) (in_bom yes) (on_board yes) (dnp no) (property "Reference" "J6" (at 294.64 119.19 0) (effects (font (size 1.2 1.2)))) (property "Value" "J6 interface" (at 294.64 134.81 0) (effects (font (size 1 1)))) (property "Footprint" "" (at 294.64 127 0) (effects (font (size 1 1)) hide)) (pin "1")(pin "2") (instances (project "nathan-controls" (path "/2f5d4a0a-9476-5e3c-a978-b6f76052ad70/a481d3d3-a1bc-5e55-a505-fd84b2acd155" (reference "J6") (unit 1)))))
+(symbol (lib_id "NATHAN:J6") (at 294.64 127 0) (unit 1) (in_bom yes) (on_board yes) (dnp no) (property "Reference" "J6" (at 294.64 119.19 0) (effects (font (size 1.2 1.2)))) (property "Value" "J6 interface" (at 294.64 134.81 0) (effects (font (size 1 1)))) (property "Footprint" "Connector_JST:JST_PH_B2B-PH-K_1x02_P2.00mm_Vertical" (at 294.64 127 0) (effects (font (size 1 1)) hide)) (pin "1")(pin "2") (instances (project "nathan-controls" (path "/2f5d4a0a-9476-5e3c-a978-b6f76052ad70/a481d3d3-a1bc-5e55-a505-fd84b2acd155" (reference "J6") (unit 1)))))
 (wire (pts (xy 276.86 127) (xy 269.24 127)) (stroke (width 0) (type default)))
 (global_label "H5_PLUS" (shape bidirectional) (at 269.24 127 0) (effects (font (size 0.9 0.9))) (property "Intersheetrefs" "${INTERSHEET_REFS}" (at 269.24 127 0) (effects (font (size 0.9 0.9)) hide)))
