File: hardware/pi3a-prototype/electrical/controls/nathan-controls.kicad_sch (KiCad schematic)
At the start: 0 parts

Commit message: feat(hardware): figer le checkpoint D1-3 et sa reprise en pause
Other:
- note added: "D1 proposal: see validation/native-current for revision-specific evidence. Component and manufacturing qualification pending."
- note removed: "D1 proposal: see validation/native-current for ERC evidence. USB/audio boundaries unresolved; no fabrication approval."
