File: hardware/pi3a-prototype/electrical/controls/power.kicad_sch (KiCad schematic)
At the start: 6 parts

Commit message: feat(hardware): figer le checkpoint D1-3 et sa reprise en pause
Parts:
- L1: value 1uH XFL3012-102ME candidate -> 1uH XAL4020-102MEC candidate; footprint (none) -> Inductor_SMD:L_Coilcraft_XAL4020-XXX
Changed lines of the file:
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@@
 (wire (pts (xy 119.38 63.5) (xy 127 63.5)) (stroke (width 0) (type default)))
 (global_label "GND" (shape bidirectional) (at 127 63.5 180) (effects (font (size 0.9 0.9))) (property "Intersheetrefs" "${INTERSHEET_REFS}" (at 127 63.5 180) (effects (font (size 0.9 0.9)) hide)))
-(symbol (lib_id "NATHAN:L1") (at 294.64 60.96 0) (unit 1) (in_bom yes) (on_board yes) (dnp no) (property "Reference" "L1" (at 294.64 53.15 0) (effects (font (size 1.2 1.2)))) (property "Value" "1uH XFL3012-102ME candidate" (at 294.64 68.77 0) (effects (font (size 1 1)))) (property "Footprint" "" (at 294.64 60.96 0) (effects (font (size 1 1)) hide)) (pin "1")(pin "2") (instances (project "nathan-controls" (path "/2f5d4a0a-9476-5e3c-a978-b6f76052ad70/9e74ff15-340f-5f3e-8810-2012facb9e33" (reference "L1") (unit 1)))))
+(symbol (lib_id "NATHAN:L1") (at 294.64 60.96 0) (unit 1) (in_bom yes) (on_board yes) (dnp no) (property "Reference" "L1" (at 294.64 53.15 0) (effects (font (size 1.2 1.2)))) (property "Value" "1uH XAL4020-102MEC candidate" (at 294.64 68.77 0) (effects (font (size 1 1)))) (property "Footprint" "Inductor_SMD:L_Coilcraft_XAL4020-XXX" (at 294.64 60.96 0) (effects (font (size 1 1)) hide))(property "Datasheet" "https://www.coilcraft.com/getmedia/6adcb47d-8b55-416c-976e-1e22e0d2848c/xal4000.pdf" (at 294.64 60.96 0) (effects (font (size 1 1)) hide)) (pin "1")(pin "2") (instances (project "nathan-controls" (path "/2f5d4a0a-9476-5e3c-a978-b6f76052ad70/9e74ff15-340f-5f3e-8810-2012facb9e33" (reference "L1") (unit 1)))))
 (wire (pts (xy 276.86 60.96) (xy 269.24 60.96)) (stroke (width 0) (type default)))
 (global_label "HAPTIC_SW" (shape bidirectional) (at 269.24 60.96 0) (effects (font (size 0.9 0.9))) (property "Intersheetrefs" "${INTERSHEET_REFS}" (at 269.24 60.96 0) (effects (font (size 0.9 0.9)) hide)))
